File: PCB/Tinylab_proto1.sch (KiCad schematic (older format))
At the start: 75 parts, among them IC1 ATXMEGA16A4U-A, P1 SCOPE_IN_CH1, P10 CONN_01X03, P11 CONN_01X03, P12 CONN_01X02, P2 USB_OTG, P3 DIG_OUT, P4 PDI, P5 SCOPE_IN_CH2, P6 DAC_OUT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

Commit message: Another Eschema Update
Have changed pinout of scope.
Still haven't added SMD pads for inductor/diode since the Element14 is
not playing ball.
Parts:
- removed P1: SCOPE_IN_CH1, Pin_Headers:Pin_Header_Straight_1x02, symbol CONN_01X02
- removed P12: CONN_01X02, Pin_Headers:Pin_Header_Straight_1x02, symbol CONN_01X02
- removed P5: SCOPE_IN_CH2, Pin_Headers:Pin_Header_Straight_1x02, symbol CONN_01X02
- removed P9: SCOPE_IN_AC, Pin_Headers:Pin_Header_Straight_1x02, symbol CONN_01X02
- added P1, P5: CONN_01X04, Pin_Headers:Pin_Header_Straight_2x04, symbol CONN_01X04
Connections:
- net at C1.1, R1.2: now also P1.1 (P1), P1.3 (P3), P1.4 (P4)
- net at C2.1, R2.2: now also P5.1 (P1), P5.3 (P3), P5.4 (P4)
- net at C2.2: now also P5.2 (P2)
- net at C1.2: now also P1.2 (P2)
Other:
- moved on the sheet: C1, C2
Changed lines of the file:
@@
 L C_Small C2
 U 1 1 55CAB4DE
-P 1700 9700
-F 0 "C2" H 1710 9770 50  0000 L CNN
-F 1 "C" H 1710 9620 50  0000 L CNN
-F 2 "Capacitors_SMD:C_0603" H 1700 9700 60  0001 C CNN
-F 3 "" H 1700 9700 60  0000 C CNN
-	1    1700 9700
+P 1550 9950
+F 0 "C2" H 1560 10020 50  0000 L CNN
+F 1 "C" H 1560 9870 50  0000 L CNN
+F 2 "Capacitors_SMD:C_0603" H 1550 9950 60  0001 C CNN
+F 3 "" H 1550 9950 60  0000 C CNN
+	1    1550 9950
 	0    1    1    0
 $EndComp
@@
 L C_Small C1
 U 1 1 55CAB611
-P 1700 9500
-F 0 "C1" H 1710 9570 50  0000 L CNN
-F 1 "C" H 1710 9420 50  0000 L CNN
-F 2 "Capacitors_SMD:C_0603" H 1700 9500 60  0001 C CNN
-F 3 "" H 1700 9500 60  0000 C CNN
-	1    1700 9500
+P 1450 9300
+F 0 "C1" H 1460 9370 50  0000 L CNN
+F 1 "C" H 1460 9220 50  0000 L CNN
+F 2 "Capacitors_SMD:C_0603" H 1450 9300 60  0001 C CNN
+F 3 "" H 1450 9300 60  0000 C CNN
+	1    1450 9300
 	0    1    1    0
 $EndComp
@@
 PSU\n
 $Comp
-L +5V #PWR01
+L +5V #PWR1
 U 1 1 55CD51C0
 P 2700 6650
-F 0 "#PWR01" H 2700 6500 50  0001 C CNN
+F 0 "#PWR1" H 2700 6500 50  0001 C CNN
 F 1 "+5V" H 2700 6790 50  0000 C CNN
 F 2 "" H 2700 6650 60  0000 C CNN
@@
 TO_B1
 $Comp
-L +5V #PWR02
+L +5V #PWR2
 U 1 1 56E7FFFF
 P 9100 5050
-F 0 "#PWR02" H 9100 4900 50  0001 C CNN
+F 0 "#PWR2" H 9100 4900 50  0001 C CNN
 F 1 "+5V" H 9100 5190 50  0000 C CNN
 F 2 "" H 9100 5050 60  0000 C CNN
@@
 	1    10000 11400
 	1    0    0    -1
-$EndComp
-$Comp
-L CONN_01X02 P1
-U 1 1 56EA2C80
-P 1200 9250
-F 0 "P1" H 1200 9400 50  0000 C CNN
-F 1 "SCOPE_IN_CH1" V 1300 9250 50  0000 C CNN
-F 2 "Pin_Headers:Pin_Header_Straight_1x02" H 1200 9250 60  0001 C CNN
-F 3 "" H 1200 9250 60  0000 C CNN
-	1    1200 9250
-	-1   0    0    1
-$EndComp
-$Comp
-L CONN_01X02 P9
-U 1 1 56EA2D2D
-P 1400 9600
-F 0 "P9" H 1400 9750 50  0000 C CNN
-F 1 "SCOPE_IN_AC" V 1500 9600 50  0000 C CNN
-F 2 "Pin_Headers:Pin_Header_Straight_1x02" H 1400 9600 60  0001 C CNN
-F 3 "" H 1400 9600 60  0000 C CNN
-	1    1400 9600
-	-1   0    0    1
-$EndComp
-$Comp
-L CONN_01X02 P5
-U 1 1 56EA3310
-P 1200 9950
-F 0 "P5" H 1200 10100 50  0000 C CNN
-F 1 "SCOPE_IN_CH2" V 1300 9950 50  0000 C CNN
-F 2 "Pin_Headers:Pin_Header_Straight_1x02" H 1200 9950 60  0001 C CNN
-F 3 "" H 1200 9950 60  0000 C CNN
-	1    1200 9950
-	-1   0    0    1
 $EndComp
 $Comp
@@
 	1    0    0    -1
 $EndComp
+NoConn ~ 13200 4850
+$Comp
+L CONN_01X04 P1
+U 1 1 5832064B
+P 1050 9250
+F 0 "P1" H 1050 9500 50  0000 C CNN
+F 1 "CONN_01X04" V 1150 9250 50  0000 C CNN
+F 2 "Pin_Headers:Pin_Header_Straight_2x04" H 1050 9250 50  0001 C CNN
+F 3 "" H 1050 9250 50  0000 C CNN
+	1    1050 9250
+	-1   0    0    1
+$EndComp
+$Comp
+L CONN_01X04 P5
+U 1 1 58320706
+P 1050 9900
+F 0 "P5" H 1050 10150 50  0000 C CNN
+F 1 "CONN_01X04" V 1150 9900 50  0000 C CNN
+F 2 "Pin_Headers:Pin_Header_Straight_2x04" H 1050 9900 50  0001 C CNN
+F 3 "" H 1050 9900 50  0000 C CNN
+	1    1050 9900
+	-1   0    0    1
+$EndComp
 Connection ~ 13950 5050
 Connection ~ 14450 5650
@@
 Connection ~ 9600 9250
 Connection ~ 10000 11550
-Connection ~ 1400 9950
-Wire Wire Line
-	1400 9900 1400 10000
-Wire Wire Line
-	1800 9950 1800 9700
-Wire Wire Line
-	1400 9950 1850 9950
-Connection ~ 1400 9250
-Wire Wire Line
-	1400 9200 1400 9300
-Wire Wire Line
-	1400 9250 1850 9250
 Wire Wire Line
 	6000 6600 6000 7100
@@
 Connection ~ 2850 9600
 Connection ~ 2350 9600
-Wire Wire Line
-	1600 9650 1600 9700
-Wire Wire Line
-	1600 9550 1600 9500
-Wire Wire Line
-	1800 9500 1800 9250
-Connection ~ 1800 9250
-Connection ~ 1800 9950
 Wire Wire Line
 	3700 8850 3700 9000
@@
 Wire Wire Line
 	13950 5300 13950 5050
-$Comp
-L CONN_01X02 P12
-U 1 1 5837E9FB
-P 13750 5350
-F 0 "P12" H 13750 5500 50  0000 C CNN
-F 1 "CONN_01X02" V 13850 5350 50  0000 C CNN
-F 2 "Pin_Headers:Pin_Header_Straight_1x02" H 13750 5350 50  0001 C CNN
-F 3 "" H 13750 5350 50  0000 C CNN
-	1    13750 5350
-	1    0    0    -1
-$EndComp
-Wire Wire Line
-	13550 5300 13550 5650
-Connection ~ 13550 5650
-Connection ~ 13550 5400
 Wire Wire Line
 	13050 4950 13200 4950
-NoConn ~ 13200 4850
+Wire Wire Line
+	1850 9100 1850 9400
+Wire Wire Line
+	1850 9100 1250 9100
+Wire Wire Line
+	1250 9200 1850 9200
+Connection ~ 1850 9200
+Wire Wire Line
+	1850 9400 1250 9400
+Connection ~ 1850 9250
+Wire Wire Line
+	1250 9300 1350 9300
+Wire Wire Line
+	1550 9300 1850 9300
+Connection ~ 1850 9300
+Wire Wire Line
+	1850 9950 1650 9950
+Wire Wire Line
+	1450 9950 1250 9950
+Wire Wire Line
+	1850 9750 1850 10050
+Wire Wire Line
+	1850 10050 1250 10050
+Wire Wire Line
+	1250 9850 1850 9850
+Connection ~ 1850 9950
+Wire Wire Line
+	1250 9750 1850 9750
+Connection ~ 1850 9850
 $EndSCHEMATC

Commit message: Error fix from last eschema
Accidentally set 2x4 headers rather than 1x4.  This has been fixed.
Parts:
- P1, P5: footprint Pin_Headers:Pin_Header_Straight_2x04 -> Pin_Headers:Pin_Header_Straight_1x04
Changed lines of the file:
@@
 PSU\n
 $Comp
-L +5V #PWR1
+L +5V #PWR01
 U 1 1 55CD51C0
 P 2700 6650
-F 0 "#PWR1" H 2700 6500 50  0001 C CNN
+F 0 "#PWR01" H 2700 6500 50  0001 C CNN
 F 1 "+5V" H 2700 6790 50  0000 C CNN
 F 2 "" H 2700 6650 60  0000 C CNN
@@
 TO_B1
 $Comp
-L +5V #PWR2
+L +5V #PWR02
 U 1 1 56E7FFFF
 P 9100 5050
-F 0 "#PWR2" H 9100 4900 50  0001 C CNN
+F 0 "#PWR02" H 9100 4900 50  0001 C CNN
 F 1 "+5V" H 9100 5190 50  0000 C CNN
 F 2 "" H 9100 5050 60  0000 C CNN
@@
 F 0 "P1" H 1050 9500 50  0000 C CNN
 F 1 "CONN_01X04" V 1150 9250 50  0000 C CNN
-F 2 "Pin_Headers:Pin_Header_Straight_2x04" H 1050 9250 50  0001 C CNN
+F 2 "Pin_Headers:Pin_Header_Straight_1x04" H 1050 9250 50  0001 C CNN
 F 3 "" H 1050 9250 50  0000 C CNN
 	1    1050 9250
@@
 F 0 "P5" H 1050 10150 50  0000 C CNN
 F 1 "CONN_01X04" V 1150 9900 50  0000 C CNN
-F 2 "Pin_Headers:Pin_Header_Straight_2x04" H 1050 9900 50  0001 C CNN
+F 2 "Pin_Headers:Pin_Header_Straight_1x04" H 1050 9900 50  0001 C CNN
 F 3 "" H 1050 9900 50  0000 C CNN
 	1    1050 9900

Commit message: Named headers
Also there's now an empty kicad_pcb file.
Parts:
- P1, P5: value CONN_01X04 -> SCOPE_OUT
- P10: value CONN_01X03 -> EXPANSION
- P11: value CONN_01X03 -> SWITCH
- P4: value PDI -> PDI/3V3
- P7: value CONN_01X02 -> PSU
Changed lines of the file:
@@
 P 4600 4350
 F 0 "P4" H 4600 4500 50  0000 C CNN
-F 1 "PDI" H 4600 4200 50  0000 C CNN
+F 1 "PDI/3V3" H 4600 4200 50  0000 C CNN
 F 2 "Pin_Headers:Pin_Header_Straight_2x02" H 4600 3150 60  0001 C CNN
 F 3 "" H 4600 3150 60  0000 C CNN
@@
 P 14150 5350
 F 0 "P7" H 14150 5500 50  0000 C CNN
-F 1 "CONN_01X02" V 14250 5350 50  0000 C CNN
+F 1 "PSU" V 14250 5350 50  0000 C CIN
 F 2 "Pin_Headers:Pin_Header_Straight_1x02" H 14150 5350 50  0001 C CNN
 F 3 "" H 14150 5350 50  0000 C CNN
@@
 P 12800 4950
 F 0 "P10" H 12800 5150 50  0000 C CNN
-F 1 "CONN_01X03" V 12900 4950 50  0000 C CNN
+F 1 "EXPANSION" V 12900 4950 50  0000 C CNN
 F 2 "Pin_Headers:Pin_Header_Straight_1x03" H 12800 4950 50  0001 C CNN
 F 3 "" H 12800 4950 50  0000 C CNN
@@
 P 13400 4950
 F 0 "P11" H 13400 5150 50  0000 C CNN
-F 1 "CONN_01X03" V 13500 4950 50  0000 C CNN
+F 1 "SWITCH" V 13500 4950 50  0000 C CNN
 F 2 "Pin_Headers:Pin_Header_Straight_1x03" H 13400 4950 50  0001 C CNN
 F 3 "" H 13400 4950 50  0000 C CNN
@@
 P 1050 9250
 F 0 "P1" H 1050 9500 50  0000 C CNN
-F 1 "CONN_01X04" V 1150 9250 50  0000 C CNN
+F 1 "SCOPE_OUT" V 1150 9250 50  0000 C CNN
 F 2 "Pin_Headers:Pin_Header_Straight_1x04" H 1050 9250 50  0001 C CNN
 F 3 "" H 1050 9250 50  0000 C CNN
@@
 P 1050 9900
 F 0 "P5" H 1050 10150 50  0000 C CNN
-F 1 "CONN_01X04" V 1150 9900 50  0000 C CNN
+F 1 "SCOPE_OUT" V 1150 9900 50  0000 C CNN
 F 2 "Pin_Headers:Pin_Header_Straight_1x04" H 1050 9900 50  0001 C CNN
 F 3 "" H 1050 9900 50  0000 C CNN
